Commit message: feat(arm_controller, mapper, ik_motion_planner): establish straight-arm zero reference and home posture
- Add rpy="-2.00719 0 0" to elbow_joint origin in arm_cad.urdf.xacro so q=[0]*6 represents a collinear vertical flagpole
- Set hardcoded home posture q=[0.0, 0.0, 2.0072, 0.0, 0.0, 0.0] corresponding to nominal resting pose (r=0.70m, z=0.22m)
- Update test_with_keyboard.py current_joints to home posture for instant RViz visual alignment
- Update ps5_mapper.py HOME_POSITIONS, FK transform chain, and world_pitch calculation
- Seed ik_solver_node.cpp with home posture and publish initial command on startup
- Update arm.srdf group_state home

File: src/arm_controller/urdf/arm_cad.urdf.xacro (robot description, xacro)
@@ -118,5 +118,6 @@
     <parent link="elbow_fixed_link" />
     <child link="elbow_link" />
-    <origin xyz="-0.047 0.000022 0.000039" rpy="0 0 0" />
+    <!-- rpy aligns Link 2 (forearm) collinearly with Link 1 (upper arm) at elbow=0 -->
+    <origin xyz="-0.047 0.000022 0.000039" rpy="-2.00719 0 0" />
     <axis xyz="1 0 0" />
     <limit lower="-2.50" upper="2.50" effort="100" velocity="1" />

Commit message: feat(arm_controller): add wrist_center frame, update elbow limits, and remove camera in URDF
- Add fixed wrist_center joint and link at Link 2 tip for decoupled 3-DOF wrist IK solving
- Set elbow_joint lower limit to 0.0 rad to prevent non-physical backward bending
- Remove extraneous RealSense camera and optical frame attachments from arm model

File: src/arm_controller/urdf/arm_cad.urdf.xacro (robot description, xacro)
@@ -1,5 +1,4 @@
 <?xml version="1.0"?>
 <robot xmlns:xacro="http://www.ros.org/wiki/xacro" name="arm">
-<xacro:include filename="$(find realsense2_description)/urdf/_d435i.urdf.xacro"/>
 <xacro:arg name="use_mock_hardware" default="false"/>
 <xacro:arg name="use_gazebo" default="false"/>
@@ -121,5 +120,5 @@
     <origin xyz="-0.047 0.000022 0.000039" rpy="-2.00719 0 0" />
     <axis xyz="1 0 0" />
-    <limit lower="-2.50" upper="2.50" effort="100" velocity="1" />
+    <limit lower="0.0" upper="2.50" effort="100" velocity="1" />
   </joint>
   <link name="bevel_link">
@@ -146,4 +145,11 @@
     <limit lower="-1.57" upper="1.57" effort="100" velocity="1" />
   </joint>
+  <!-- Wrist pitch axis center frame for decoupled 3-DOF positioning -->
+  <joint name="wrist_center_joint" type="fixed">
+    <parent link="bevel_link" />
+    <child link="wrist_center" />
+    <origin xyz="0 -0.117291 -0.054694" rpy="0 0 0" />
+  </joint>
+  <link name="wrist_center" />
   <link name="wrist_pitch_link">
     <visual>
@@ -193,15 +199,4 @@
   </joint>
   <link name="tool0"/>
-  <!-- ========================= -->
-  <!-- Intel RealSense D435i Mount -->
-  <!-- ========================= -->
-  <xacro:sensor_d435i
-    parent="gripper_link"
-    name="camera"
-    use_nominal_extrinsics="true">
-    <origin
-        xyz="0 0.03 0.07"
-        rpy="0 0 ${PI/2}"/>
-  </xacro:sensor_d435i>
   <link name="upper_jaw_link">
     <visual>
@@ -270,25 +265,4 @@
   </plugin>
 </gazebo>
-<gazebo reference="camera_link">
-  <sensor name="d435i_rgbd" type="rgbd_camera">
-    <always_on>true</always_on>
-    <visualize>true</visualize>
-    <update_rate>30</update_rate>
-    <topic>camera</topic>
-    <gz_frame_id>camera_link</gz_frame_id>
-    <camera>
-      <horizontal_fov>1.211</horizontal_fov>
-      <camera_info_topic>camera/camera_info</camera_info_topic>
-      <image>
-        <width>1920</width>
-        <height>1080</height>
-        <format>R8G8B8</format>
-      </image>
-      <clip>
-        <near>0.1</near>
-        <far>10.0</far>
-      </clip>
-    </camera>
-  </sensor>
-</gazebo>
+<!--Camera Part Removed -->
 </robot>
